File: new_pcb_main_board/design/pcb_main_board.kicad_pcb (KiCad board)
At the start: 2 copper layers, 85 x 56 mm, 75 parts, among them IC1 MP2338GTL-Z, IC2 MP2338GTL-Z, J1 Conn_01x02_Socket, J2 PWM1, J4 PWM2, J5 PWM3, J6 PWM4, J7 MOT_A, J8 MOT_B, J9 Conn_02x20_Odd_Even, SW1 SW_Push, U1 CH32V003FxUx, U3 TB6612FNG

Commit message: PCB rev2 update
Parts:
- removed C16: 470uF, Capacitor_THT:CP_Radial_D8.0mm_P3.50mm
- removed H5: MountingVia1, MountingHole:MountingHole_3.2mm_M3_Pad_Via
- removed H6: MountingVia2, MountingHole:MountingHole_3.2mm_M3_Pad_Via
- removed H7: MountingVia3, MountingHole:MountingHole_3.2mm_M3_Pad_Via
- removed U1: CH32V003FxUx, Package_DFN_QFN:QFN-20-1EP_3x3mm_P0.4mm_EP1.65x1.65mm
- added G***: LOGO, CustomIcon:PiCarIcon, F.Cu at (210.2, 81.3)
- added U2: CH32V003AxMx, Package_SO:STC_SOP-16_3.9x9.9mm_P1.27mm, F.Cu at (224.0, 89.0)
- C10, C13, C17, C19, C2, C20, C21, C23, C26, C27, C3, C4, C5, C6, C7, C8, C9: footprint Capacitor_SMD:C_0805_2012Metric_Pad1.18x1.45mm_HandSolder -> Capacitor_SMD:C_0805_2012Metric
- R1, R10, R11, R12, R13, R14, R15, R19, R2, R20, R21, R22, R23, R24, R3, R4, R6, R7, R8, R9: footprint Resistor_SMD:R_0805_2012Metric_Pad1.20x1.40mm_HandSolder -> Resistor_SMD:R_0805_2012Metric
- moved C10 40.1 mm to (186.7, 104.1), turned to 180 degrees
- moved J8 38.6 mm to (190.4, 122.5), turned to 0 degrees
- moved C3 37.1 mm to (164.5, 95.5), turned to 180 degrees
- moved C2 37.1 mm to (164.5, 93.5), turned to 180 degrees
- moved C4 37.1 mm to (164.5, 97.5), turned to 180 degrees
- moved C9 35.8 mm to (186.7, 106.1), turned to 180 degrees
- moved C14 35.6 mm to (163.7, 119.5)
- moved C15 35.6 mm to (163.7, 121.5)
- moved L1 35.6 mm to (155.5, 105.9), turned to -90 degrees
- moved J7 34.7 mm to (178.4, 122.5), turned to 0 degrees
- moved R5 33.7 mm to (231.5, 91.5), turned to 180 degrees
- moved H4 32.8 mm to (162.5, 124.5)
- moved C12 27.2 mm to (224.0, 81.7), turned to 180 degrees
- moved C11 26.3 mm to (224.0, 79.6), turned to 180 degrees
- moved D2 26.1 mm to (232.0, 84.8), turned to -90 degrees
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Connections:
- net Net-(C18-Pad2) renamed /BAT_ADC
- net Net-(C25-Pad1) renamed /NRST
- J9 pad 9: unconnected-(J9-Pin_9-Pad9) -> GND
- R20 pad 1: unconnected-(R20-Pad1) -> /LED
Routing:
- net +BATT: track 0.00 -> 129.9 mm
- net GND: track 0.00 -> 53.9 mm, vias 0 -> 44
- net /4V8: track 0.00 -> 31.1 mm
- net /5V1: track 0.00 -> 27.3 mm
- net +3V3: track 0.00 -> 15.3 mm
- net /NRST: track 0.00 -> 11.9 mm
- net Net-(IC1-EN): track 0.00 -> 10.5 mm
- net Net-(J8-Pin_2): track 0.00 -> 8.54 mm
- net Net-(J7-Pin_1): track 0.00 -> 8.35 mm
- net Net-(J8-Pin_1): track 0.00 -> 7.56 mm
- net Net-(J7-Pin_2): track 0.00 -> 7.33 mm
- net Net-(C17-Pad1): track 0.00 -> 7.11 mm
- net Net-(C27-Pad1): track 0.00 -> 6.60 mm
- net Net-(IC2-SW): track 0.00 -> 5.74 mm
- net /LED: track 0.00 -> 5.57 mm
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- added copper zone on B.Cu, net GND
Other:
- outline, holes or cut-outs redrawn
- board text added: "24.07.2026"
- board text added: "Mateusz Antkiewicz"
- board text added: "PiCar"
- board text added: "rev 2"
