File: new_pcb_main_board/design/pcb_main_board.kicad_sch (KiCad schematic)
At the start: 75 parts, among them IC1 MP2338GTL-Z, IC2 MP2338GTL-Z, J1 Conn_01x02_Socket, J2 PWM1, J4 PWM2, J5 PWM3, J6 PWM4, J7 MOT_A, J8 MOT_B, J9 Conn_02x20_Odd_Even, SW1 SW_Push, U1 CH32V003FxUx, U3 TB6612FNG

Commit message: PCB rev2 update
Parts:
- removed C16: 470uF, Capacitor_THT:CP_Radial_D8.0mm_P3.50mm, symbol Device:C_Polarized
- removed H5: MountingVia1, MountingHole:MountingHole_3.2mm_M3_Pad_Via, symbol Mechanical:MountingHole_Pad
- removed H6: MountingVia2, MountingHole:MountingHole_3.2mm_M3_Pad_Via, symbol Mechanical:MountingHole_Pad
- removed H7: MountingVia3, MountingHole:MountingHole_3.2mm_M3_Pad_Via, symbol Mechanical:MountingHole_Pad
- removed U1: CH32V003FxUx, Package_DFN_QFN:QFN-20-1EP_3x3mm_P0.4mm_EP1.65x1.65mm, symbol MCU_WCH_RiscV:CH32V003FxUx
- added U2: CH32V003AxMx, Package_SO:STC_SOP-16_3.9x9.9mm_P1.27mm, symbol MCU_WCH_RiscV:CH32V003AxMx
- C10, C13, C17, C19, C2, C20, C21, C23, C26, C27, C3, C4, C5, C6, C7, C8, C9: footprint Capacitor_SMD:C_0805_2012Metric_Pad1.18x1.45mm_HandSolder -> Capacitor_SMD:C_0805_2012Metric
- R1, R10, R11, R12, R13, R14, R15, R19, R2, R20, R21, R22, R23, R24, R3, R4, R6, R7, R8, R9: footprint Resistor_SMD:R_0805_2012Metric_Pad1.20x1.40mm_HandSolder -> Resistor_SMD:R_0805_2012Metric
Connections:
- net +3V3: now also U2.15 (VDD)
- net DIR1: now also U2.8 (PD4)
- net DIR2: now also U2.16 (PC0)
- net GND: now also J9.9 (Pin_9), U2.14 (VSS)
- net SCL: now also U2.2 (PC2)
- net SDA: now also U2.1 (PC1)
- net SWDIO: now also U2.7 (PD1)
- net T1CH1_1: now also U2.5 (PC6)
- net T1CH2_1: now also U2.6 (PC7)
- net T1CH3: now also U2.3 (PC3)
- net T1CH4: now also U2.4 (PC4)
- net T2CH3_3: now also U2.10 (PD6)
- net T2CH4_3: now also U2.9 (PD5)
- net LED: now reaches R20.1
- net LED: now also U2.12 (PA1)
- net NRST: now reaches C25.1, R5.2, SW1.1
- net NRST: now also U2.11 (PD7)
- net BAT_ADC: now reaches C18.2, R17.2
- net BAT_ADC: now also U2.13 (PA2)
Other:
- moved on the sheet: C18, D2, J1, R16, R17, R18, R20
